Commit message: tried using xacro properties to fix mesh position to joints and added virtual claw

File: theseus_description/urdf/theseus_real.urdf.xacro (robot description, xacro)
@@ -4,4 +4,25 @@
     <xacro:property name="effort" value="10.0"/>
     <xacro:property name="velocity" value="5.0"/>
+    <!-- Claw -->
+    <xacro:property name="finger_length" value="0.15"/>
+    <!-- Mesh scale -->
+    <xacro:property name="mesh_scale" value="0.003 0.003 0.003"/>
+    <!-- Joint distances -->
+    <!-- They are relative to one another eg. arm_joint_2 distances are relative to arm_joint_1 position -->
+    <xacro:property name="base_arm_joint_x" value="0.0"/>
+    <xacro:property name="base_arm_joint_y" value="0.0"/>
+    <xacro:property name="base_arm_joint_z" value="0.0"/>
+    <xacro:property name="arm_joint_1_x" value="0.0"/>
+    <xacro:property name="arm_joint_1_y" value="0.0"/>
+    <xacro:property name="arm_joint_1_z" value="0.31"/>
+    <xacro:property name="arm_joint_2_x" value="0.0"/>
+    <xacro:property name="arm_joint_2_y" value="0.0"/>
+    <xacro:property name="arm_joint_2_z" value="0.75"/>
+    <xacro:property name="arm_joint_3_x" value="0.0"/>
+    <xacro:property name="arm_joint_3_y" value="-0.225"/>
+    <xacro:property name="arm_joint_3_z" value="0.485"/>
+    <xacro:property name="arm_joint_4_x" value="0.0"/>
+    <xacro:property name="arm_joint_4_y" value="-0.25"/>
+    <xacro:property name="arm_joint_4_z" value="-0.91"/>
     <link name="world"/>
     <link name="base_link">
@@ -9,5 +30,5 @@
             <origin rpy="0 0 0" xyz="-0.015 0 0.38"/>
             <geometry>
-                <mesh filename="package://manipulator_description/meshes/theseus_link_1.stl" scale="0.003 0.003 0.003"/>
+                <mesh filename="package://manipulator_description/meshes/theseus_link_1.stl" scale="${mesh_scale}"/>
             </geometry>
         </visual>
@@ -20,7 +41,8 @@
     <link name="arm_link_1">
         <visual>
-            <origin rpy="0 0 0" xyz="0 0 0.075"/>
+            <!-- 0 0 0.075 -->
+            <origin rpy="0 0 0" xyz="${arm_joint_1_x} ${arm_joint_1_y} ${arm_joint_1_z-0.235}"/>
             <geometry>
-                <mesh filename="package://manipulator_description/meshes/theseus_link_2.stl" scale="0.003 0.003 0.003"/>
+                <mesh filename="package://manipulator_description/meshes/theseus_link_2.stl" scale="${mesh_scale}"/>
             </geometry>
         </visual>
@@ -30,12 +52,13 @@
         <child link="arm_link_1"/>
         <axis xyz="1 0 0"/>
-        <origin rpy="0 0 0" xyz="0 0 0.31"/>
+        <origin rpy="0 0 0" xyz="${arm_joint_1_x} ${arm_joint_1_y} ${arm_joint_1_z}"/>
         <limit lower="-${PI/2}" upper="${PI/2}" effort="${effort}" velocity="${velocity}"/>
     </joint>
     <link name="arm_link_2">
         <visual>
-            <origin rpy="0 0 0" xyz="0 0 -0.66"/>
+            <!-- 0 0 -0.66 -->
+            <origin rpy="0 0 0" xyz="${arm_joint_2_x} ${arm_joint_2_y} ${arm_joint_2_z-1.41}"/>
             <geometry>
-                <mesh filename="package://manipulator_description/meshes/theseus_link_3.stl" scale="0.003 0.003 0.003"/>
+                <mesh filename="package://manipulator_description/meshes/theseus_link_3.stl" scale="${mesh_scale}"/>
             </geometry>
         </visual>
@@ -45,12 +68,13 @@
         <child link="arm_link_2"/>
         <axis xyz="0 0 1"/>
-        <origin rpy="0 0 0" xyz="0 0 0.75"/>
+        <origin rpy="0 0 0" xyz="${arm_joint_2_x} ${arm_joint_2_y} ${arm_joint_2_z}"/>
         <limit lower="-${PI/2}" upper="${PI/2}" effort="${effort}" velocity="${velocity}"/>
     </joint>
     <link name="arm_link_3">
         <visual>
-            <origin rpy="0 0 0" xyz="0 0.22 -1.15"/>
+            <!-- 0 0.22 -1.15 -->
+            <origin rpy="0 0 0" xyz="${arm_joint_3_x} ${arm_joint_3_y+0.445} ${arm_joint_3_z-1.635} 0.22 -1.15"/>
             <geometry>
-                <mesh filename="package://manipulator_description/meshes/theseus_link_4.stl" scale="0.003 0.003 0.003"/>
+                <mesh filename="package://manipulator_description/meshes/theseus_link_4.stl" scale="${mesh_scale}"/>
             </geometry>
         </visual>
@@ -60,12 +84,13 @@
         <child link="arm_link_3"/>
         <axis xyz="1 0 0"/>
-        <origin rpy="0 0 0" xyz="0 -0.225 0.485"/>
+        <origin rpy="0 0 0" xyz="${arm_joint_3_x} ${arm_joint_3_y} ${arm_joint_3_z}"/>
         <limit lower="-${PI/2}" upper="${PI/2}" effort="${effort}" velocity="${velocity}"/>
     </joint>
     <link name="arm_link_4">
         <visual>
-            <origin rpy="0 0 0" xyz="0 0.47 -0.24"/>
+            <!-- 0 0.47 -0.24 -->
+            <origin rpy="0 0 0" xyz="${arm_joint_4_x} ${arm_joint_4_y+0.72} ${arm_joint_4_z+0.67}"/>
             <geometry>
-                <mesh filename="package://manipulator_description/meshes/theseus_link_5.stl" scale="0.003 0.003 0.003"/>
+                <mesh filename="package://manipulator_description/meshes/theseus_link_5.stl" scale="${mesh_scale}"/>
             </geometry>
         </visual>
@@ -75,7 +100,49 @@
         <child link="arm_link_4"/>
         <axis xyz="1 0 0"/>
-        <origin rpy="0 0 0" xyz="0 -0.25 -0.91"/>
+        <origin rpy="0 0 0" xyz="${arm_joint_4_x} ${arm_joint_4_y} ${arm_joint_4_z}"/>
         <limit lower="-${PI/2}" upper="${PI/2}" effort="${effort}" velocity="${velocity}"/>
+    <!-- Not the real claw -->
+    <link name="gripper_right">
+        <visual>
+            <origin rpy="0 0 -${PI/2}" xyz="0 -0.02 ${finger_length/2}"/>
+            <geometry>
+                <cylinder radius="0.02" length="${finger_length}"/>
+            </geometry>
+        </visual>
+        <collision>
+            <origin rpy="0 0 -${PI/2}" xyz="0 -0.02 ${finger_length/2}"/>
+            <geometry>
+                <cylinder radius="0.02" length="${finger_length}"/>
+            </geometry>
+        </collision>
+    </link>
+    <link name="gripper_left">
+        <visual>
+            <origin rpy="0 0 -${PI/2}" xyz="0 0.02 ${finger_length/2}"/>
+            <geometry>
+                <cylinder radius="0.02" length="${finger_length}"/>
+            </geometry>
+        </visual>
+        <collision>
+            <origin rpy="0 0 -${PI/2}" xyz="0 -0.02 ${finger_length/2}"/>
+            <geometry>
+                <cylinder radius="0.02" length="${finger_length}"/>
+            </geometry>
+        </collision>
+    </link>
+    <joint name="gripper_joint_1" type="revolute">
+        <parent link="arm_joint_4"/>
+        <child link="gripper_right"/>
+        <axis xyz="1 0 0"/>
+        <origin rpy="0 0 0" xyz="0 0 0"/>
+        <limit lower="0" upper="${PI/2}" effort="${effort}" velocity="${velocity}"/>
     </joint>
-    <!-- Primeiro 6cm, depois 34cm, depois 27cm -->
+    <joint name="gripper_joint_2" type="revolute">
+        <parent link="arm_joint_4"/>
+        <child link="gripper_left"/>
+        <axis xyz="1 0 0"/>
+        <origin rpy="0 0 0" xyz="0 0 0"/>
+        <mimic joint="gripper_joint_1" multiplier="-1"/>
+        <limit lower="0" upper="${PI/2}" effort="${effort}" velocity="${velocity}"/>
+    </joint>
 </robot>

Commit message: Checkpoint

File: theseus_description/urdf/theseus_real.urdf.xacro (robot description, xacro)
@@ -5,5 +5,5 @@
     <xacro:property name="velocity" value="5.0"/>
     <!-- Claw -->
-    <xacro:property name="finger_length" value="0.15"/>
+    <xacro:property name="finger_length" value="0.05"/>
     <!-- Mesh scale -->
     <xacro:property name="mesh_scale" value="0.003 0.003 0.003"/>
@@ -25,4 +25,7 @@
     <xacro:property name="arm_joint_4_y" value="-0.25"/>
     <xacro:property name="arm_joint_4_z" value="-0.91"/>
+    <xacro:property name="gripper_joint_x" value="0.04"/>
+    <xacro:property name="gripper_joint_y" value="0.0"/>
+    <xacro:property name="gripper_joint_z" value="-0.22"/>
     <link name="world"/>
     <link name="base_link">
@@ -30,5 +33,5 @@
             <origin rpy="0 0 0" xyz="-0.015 0 0.38"/>
             <geometry>
-                <mesh filename="package://manipulator_description/meshes/theseus_link_1.stl" scale="${mesh_scale}"/>
+                <mesh filename="package://theseus_description/meshes/theseus_link_1.stl" scale="${mesh_scale}"/>
             </geometry>
         </visual>
@@ -44,5 +47,5 @@
             <origin rpy="0 0 0" xyz="${arm_joint_1_x} ${arm_joint_1_y} ${arm_joint_1_z-0.235}"/>
             <geometry>
-                <mesh filename="package://manipulator_description/meshes/theseus_link_2.stl" scale="${mesh_scale}"/>
+                <mesh filename="package://theseus_description/meshes/theseus_link_2.stl" scale="${mesh_scale}"/>
             </geometry>
         </visual>
@@ -60,5 +63,5 @@
             <origin rpy="0 0 0" xyz="${arm_joint_2_x} ${arm_joint_2_y} ${arm_joint_2_z-1.41}"/>
             <geometry>
-                <mesh filename="package://manipulator_description/meshes/theseus_link_3.stl" scale="${mesh_scale}"/>
+                <mesh filename="package://theseus_description/meshes/theseus_link_3.stl" scale="${mesh_scale}"/>
             </geometry>
         </visual>
@@ -74,7 +77,7 @@
         <visual>
             <!-- 0 0.22 -1.15 -->
-            <origin rpy="0 0 0" xyz="${arm_joint_3_x} ${arm_joint_3_y+0.445} ${arm_joint_3_z-1.635} 0.22 -1.15"/>
+            <origin rpy="0 0 0" xyz="${arm_joint_3_x} ${arm_joint_3_y+0.445} ${arm_joint_3_z-1.635}"/>
             <geometry>
-                <mesh filename="package://manipulator_description/meshes/theseus_link_4.stl" scale="${mesh_scale}"/>
+                <mesh filename="package://theseus_description/meshes/theseus_link_4.stl" scale="${mesh_scale}"/>
             </geometry>
         </visual>
@@ -92,5 +95,5 @@
             <origin rpy="0 0 0" xyz="${arm_joint_4_x} ${arm_joint_4_y+0.72} ${arm_joint_4_z+0.67}"/>
             <geometry>
-                <mesh filename="package://manipulator_description/meshes/theseus_link_5.stl" scale="${mesh_scale}"/>
+                <mesh filename="package://theseus_description/meshes/theseus_link_5.stl" scale="${mesh_scale}"/>
             </geometry>
         </visual>
@@ -102,16 +105,38 @@
         <origin rpy="0 0 0" xyz="${arm_joint_4_x} ${arm_joint_4_y} ${arm_joint_4_z}"/>
         <limit lower="-${PI/2}" upper="${PI/2}" effort="${effort}" velocity="${velocity}"/>
+    </joint>
     <!-- Not the real claw -->
-    <link name="gripper_right">
+    <link name="gripper_link">
         <visual>
-            <origin rpy="0 0 -${PI/2}" xyz="0 -0.02 ${finger_length/2}"/>
+            <origin rpy="0 ${PI/2} -${PI/2}" xyz="0 0 -0.05"/>
             <geometry>
-                <cylinder radius="0.02" length="${finger_length}"/>
+                <mesh filename="package://theseus_description/meshes/gripper_main_link.stl" scale="${mesh_scale}"/>
             </geometry>
         </visual>
         <collision>
-            <origin rpy="0 0 -${PI/2}" xyz="0 -0.02 ${finger_length/2}"/>
+            <origin rpy="0 ${PI/2} -${PI/2}" xyz="0 0 -0.05"/>
             <geometry>
-                <cylinder radius="0.02" length="${finger_length}"/>
+                <mesh filename="package://theseus_description/meshes/gripper_main_link.stl" scale="${mesh_scale}"/>
+            </geometry>
+        </collision>
+    </link>
+    <joint name="gripper_joint" type="revolute">
+        <parent link="arm_link_4"/>
+        <child link="gripper_link"/>
+        <axis xyz="1 0 0"/>
+        <origin rpy="0 0 0" xyz="${gripper_joint_x} ${gripper_joint_y} ${gripper_joint_z}"/>
+        <limit lower="-${PI/2}" upper="${PI/2}" effort="${effort}" velocity="${velocity}"/>
+    </joint>
+    <link name="gripper_right">
+        <visual>
+            <origin rpy="0 ${PI/2} -${PI/2}" xyz="-0 0 -${finger_length/2}"/>
+            <geometry>
+                <mesh filename="package://theseus_description/meshes/gripper_link.stl" scale="${mesh_scale}"/>
+            </geometry>
+        </visual>
+        <collision>
+            <origin rpy="0 ${PI/2} -${PI/2}" xyz="-0 0 -${finger_length/2}"/>
+            <geometry>
+                <mesh filename="package://theseus_description/meshes/gripper_link.stl" scale="${mesh_scale}"/>
             </geometry>
         </collision>
@@ -119,28 +144,28 @@
     <link name="gripper_left">
         <visual>
-            <origin rpy="0 0 -${PI/2}" xyz="0 0.02 ${finger_length/2}"/>
+            <origin rpy="0 ${PI/2} -${PI/2}" xyz="0 0 -${finger_length/2}"/>
             <geometry>
-                <cylinder radius="0.02" length="${finger_length}"/>
+                <mesh filename="package://theseus_description/meshes/gripper_sub_link.stl" scale="${mesh_scale}"/>
             </geometry>
         </visual>
         <collision>
-            <origin rpy="0 0 -${PI/2}" xyz="0 -0.02 ${finger_length/2}"/>
+            <origin rpy="0 ${PI/2} -${PI/2}" xyz="0 0 -${finger_length/2}"/>
             <geometry>
-                <cylinder radius="0.02" length="${finger_length}"/>
+                <mesh filename="package://theseus_description/meshes/gripper_sub_link.stl" scale="${mesh_scale}"/>
             </geometry>
         </collision>
     </link>
     <joint name="gripper_joint_1" type="revolute">
-        <parent link="arm_joint_4"/>
+        <parent link="gripper_link"/>
         <child link="gripper_right"/>
-        <axis xyz="1 0 0"/>
-        <origin rpy="0 0 0" xyz="0 0 0"/>
+        <axis xyz="0 1 0"/>
+        <origin rpy="0 0 0" xyz="${-gripper_joint_x} ${gripper_joint_y} ${gripper_joint_z}"/>
         <limit lower="0" upper="${PI/2}" effort="${effort}" velocity="${velocity}"/>
     </joint>
     <joint name="gripper_joint_2" type="revolute">
-        <parent link="arm_joint_4"/>
+        <parent link="gripper_link"/>
         <child link="gripper_left"/>
-        <axis xyz="1 0 0"/>
-        <origin rpy="0 0 0" xyz="0 0 0"/>
+        <axis xyz="0 1 0"/>
+        <origin rpy="0 0 0" xyz="${gripper_joint_x} ${gripper_joint_y} ${gripper_joint_z}"/>
         <mimic joint="gripper_joint_1" multiplier="-1"/>
         <limit lower="0" upper="${PI/2}" effort="${effort}" velocity="${velocity}"/>
