Commit message: WORKING FUCK YEHA simulation only though

File: theseus_description/urdf/manipulator_ros2_control.xacro (robot description, xacro)
@@ -15,5 +15,5 @@
                 </hardware>
             </xacro:unless>
-            <joint name="gripper_joint_2">
+            <!-- <joint name="gripper_joint_2">
                 <param name="mimic">gripper_joint_1</param>
                 <param name="multiplier">-1</param>
@@ -23,5 +23,5 @@
                 </command_interface>
                 <state_interface name="position"/>
-            </joint>
+            </joint>  -->
         </xacro:if>
         <!-- ros2_control real manipulator only -->

File: theseus_description/urdf/theseus.urdf.xacro (robot description, xacro)
@@ -240,11 +240,15 @@
         <limit lower="${-PI/9}" upper="${PI/2}" effort="${effort}" velocity="${velocity}"/>
     </joint>
-    <joint name="gripper_joint_2" type="revolute">
+    <joint name="gripper_joint_2_mimic" type="fixed">
         <parent link="gripper_link"/>
         <child link="gripper_left"/>
-        <axis xyz="0 1 0"/>
+        <!-- <axis xyz="0 1 0"/> -->
         <origin rpy="0 0 0" xyz="${finger_separation} 0 ${-finger_length}"/>
-        <mimic joint="gripper_joint_1" multiplier="-1"/>
-        <limit lower="${-PI/9}" upper="${PI/2}" effort="${effort}" velocity="${velocity}"/>
-    </joint>
+        <!-- <mimic joint="gripper_joint_1" multiplier="-1"/>
+        <limit lower="${-PI/9}" upper="${PI/2}" effort="${effort}" velocity="${velocity}"/> -->
+    </joint>
+    <!-- <joint name="gripper_joint_2_mimic" type="fixed">
+    <parent link="world" />
+    <child link="gripper_left" />
+    </joint> -->
 </robot>

Commit message: test code

File: theseus_description/urdf/manipulator_ros2_control.xacro (robot description, xacro)
@@ -15,5 +15,5 @@
                 </hardware>
             </xacro:unless>
-            <!-- <joint name="gripper_joint_2">
+            <joint name="gripper_joint_2">
                 <param name="mimic">gripper_joint_1</param>
                 <param name="multiplier">-1</param>
@@ -23,5 +23,5 @@
                 </command_interface>
                 <state_interface name="position"/>
-            </joint>  -->
+            </joint>
         </xacro:if>
         <!-- ros2_control real manipulator only -->
