Commit message: theseus model updated to real

File: theseus_description/urdf/manipulator.urdf.xacro (robot description, xacro)
@@ -7,5 +7,5 @@
     <xacro:include filename="$(find theseus_description)/urdf/theseus_gazebo.xacro"/>
     <!-- Include ros2_control plugins -->
-    <xacro:include filename="$(find theseus_description)/urdf/theseus_ros2_control.xacro"/>
+    <xacro:include filename="$(find theseus_description)/urdf/manipulator_ros2_control.xacro"/>
     <!-- Useful XACRO variables -->
     <xacro:property name="PI" value="3.14159265358979323846"/>

File: theseus_description/urdf/manipulator_ros2_control.xacro (robot description, xacro)
@@ -34,6 +34,6 @@
         <joint name="arm_joint_1">
             <command_interface name="position">
-            <param name="min">${-PI/2}</param>
-            <param name="max">${PI/2}</param>
+            <param name="min">-${3*PI/4}</param>
+            <param name="max">${3*PI/4}</param>
             </command_interface>
             <state_interface name="position"/>
@@ -41,27 +41,6 @@
         <joint name="arm_joint_2">
             <command_interface name="position">
-            <param name="min">${-PI/2}</param>
-            <param name="max">${PI/2}</param>
-            </command_interface>
-            <state_interface name="position"/>
-        </joint>
-        <joint name="arm_joint_3">
-            <command_interface name="position">
-            <param name="min">${-PI/2}</param>
-            <param name="max">${PI/2}</param>
-            </command_interface>
-            <state_interface name="position"/>
-        </joint>
-        <joint name="arm_joint_4">
-            <command_interface name="position">
-            <param name="min">${-PI/2}</param>
-            <param name="max">${PI/2}</param>
-            </command_interface>
-            <state_interface name="position"/>
-        </joint>
-        <joint name="gripper_joint">
-            <command_interface name="position">
-            <param name="min">${-PI/2}</param>
-            <param name="max">${PI/2}</param>
+            <param name="min">-${3*PI/4}</param>
+            <param name="max">${3*PI/4}</param>
             </command_interface>
             <state_interface name="position"/>
@@ -69,5 +48,5 @@
         <joint name="gripper_joint_1">
             <command_interface name="position">
-            <param name="min">${-PI/9}</param>
+            <param name="min">0</param>
             <param name="max">${PI/2}</param>
             </command_interface>

File: theseus_description/urdf/theseus_real.urdf.xacro (robot description, xacro)
@@ -1,9 +1,23 @@
 <?xml version="1.0"?>
 <robot xmlns:xacro="http://www.ros.org/wiki/xacro" name="utbots_manipulator">
+    <!-- Simulation flags for switching simulation engines before and after ROS2 Humble -->
+    <xacro:arg name="is_sim" default="false" />
+    <xacro:arg name="is_ignition" default="true" />
+    <!-- Include Gazebo Parameters (only relevant for sim) -->
+    <xacro:include filename="$(find theseus_description)/urdf/theseus_gazebo.xacro"/>
+    <!-- Include ros2_control plugins -->
+    <xacro:include filename="$(find theseus_description)/urdf/theseus_ros2_control.xacro"/>
+    <!-- Placeholder properties (may need changing later) -->
     <xacro:property name="PI" value="3.14159265358979323846"/>
+    <xacro:macro name="default_inertial" params="mass">
+        <inertial>
+            <mass value="${mass}"/>
+            <inertia ixx="1.0" ixy="0.0" ixz="0.0"
+                     iyy="1.0" iyz="0.0"
+                     izz="1.0"/>
+        </inertial>
+    </xacro:macro>
     <xacro:property name="effort" value="10.0"/>
     <xacro:property name="velocity" value="5.0"/>
-    <!-- Claw -->
-    <xacro:property name="finger_length" value="0.05"/>
     <!-- Mesh scale -->
     <xacro:property name="mesh_scale" value="0.003 0.003 0.003"/>
@@ -28,6 +42,9 @@
     <xacro:property name="gripper_joint_y" value="0.0"/>
     <xacro:property name="gripper_joint_z" value="-0.22"/>
+    <xacro:property name="finger_length" value="0.05"/>
+    <!-- Links and Joints -->
     <link name="world"/>
     <link name="base_link">
+        <xacro:default_inertial mass="0.2"/>
         <visual>
             <origin rpy="0 0 0" xyz="-0.015 0 0.38"/>
@@ -36,4 +53,10 @@
             </geometry>
         </visual>
+        <collision>
+            <origin rpy="0 0 0" xyz="-0.015 0 0.38"/>
+            <geometry>
+                <mesh filename="package://theseus_description/meshes/theseus_link_1.stl" scale="${mesh_scale}"/>
+            </geometry>
+        </collision>
     </link>
     <joint name="base_arm_joint" type="fixed">
@@ -43,4 +66,5 @@
     </joint>
     <link name="arm_link_1">
+        <xacro:default_inertial mass="1.0"/>
         <visual>
             <!-- 0 0 0.075 -->
@@ -50,4 +74,10 @@
             </geometry>
         </visual>
+        <collision>
+            <origin rpy="0 0 0" xyz="${arm_joint_1_x} ${arm_joint_1_y} ${arm_joint_1_z-0.235}"/>
+            <geometry>
+                <mesh filename="package://theseus_description/meshes/theseus_link_2.stl" scale="${mesh_scale}"/>
+            </geometry>
+        </collision>
     </link>
     <joint name="arm_joint_1" type="revolute">
@@ -59,4 +89,5 @@
     </joint>
     <link name="arm_link_2">
+        <xacro:default_inertial mass="0.3"/>
         <visual>
             <!-- 0 0 -0.66 -->
@@ -66,4 +97,11 @@
             </geometry>
         </visual>
+        <collision>
+            <!-- 0 0 -0.66 -->
+            <origin rpy="0 0 0" xyz="${arm_joint_2_x} ${arm_joint_2_y} ${arm_joint_2_z-1.41}"/>
+            <geometry>
+                <mesh filename="package://theseus_description/meshes/theseus_link_3.stl" scale="${mesh_scale}"/>
+            </geometry>
+        </collision>
     </link>
     <joint name="arm_joint_2" type="revolute">
@@ -75,4 +113,5 @@
     </joint>
     <link name="arm_link_3">
+        <xacro:default_inertial mass="0.5"/>
         <visual>
             <!-- 0 0.22 -1.15 -->
@@ -82,4 +121,10 @@
             </geometry>
         </visual>
+        <collision>
+            <origin rpy="0 0 0" xyz="${arm_joint_3_x} ${arm_joint_3_y+0.445} ${arm_joint_3_z-1.635}"/>
+            <geometry>
+                <mesh filename="package://theseus_description/meshes/theseus_link_4.stl" scale="${mesh_scale}"/>
+            </geometry>
+        </collision>
     </link>
     <joint name="arm_joint_3" type="revolute">
@@ -91,4 +136,5 @@
     </joint>
     <link name="arm_link_4">
+        <xacro:default_inertial mass="0.2"/>
         <visual>
             <!-- 0 0.47 -0.24 -->
@@ -98,4 +144,10 @@
             </geometry>
         </visual>
+        <collision>
+            <origin rpy="0 0 0" xyz="${arm_joint_4_x} ${arm_joint_4_y+0.72} ${arm_joint_4_z+0.67}"/>
+            <geometry>
+                <mesh filename="package://theseus_description/meshes/theseus_link_5.stl" scale="${mesh_scale}"/>
+            </geometry>
+        </collision>
     </link>
     <joint name="arm_joint_4" type="revolute">
@@ -108,4 +160,5 @@
     <!-- Not the real claw -->
     <link name="gripper_link">
+        <xacro:default_inertial mass="0.1"/>
         <visual>
             <origin rpy="0 ${PI/2} -${PI/2}" xyz="0 0 -0.05"/>
@@ -124,9 +177,10 @@
         <parent link="arm_link_4"/>
         <child link="gripper_link"/>
-        <axis xyz="1 0 0"/>
+        <axis xyz="0 0 1"/>
         <origin rpy="0 0 0" xyz="${gripper_joint_x} ${gripper_joint_y} ${gripper_joint_z}"/>
         <limit lower="-${PI/2}" upper="${PI/2}" effort="${effort}" velocity="${velocity}"/>
     </joint>
     <link name="gripper_right">
+        <xacro:default_inertial mass="0.1"/>
         <visual>
             <origin rpy="0 ${PI/2} -${PI/2}" xyz="-0 0 -${finger_length/2}"/>
@@ -143,4 +197,5 @@
     </link>
     <link name="gripper_left">
+        <xacro:default_inertial mass="0.1"/>
         <visual>
             <origin rpy="0 ${PI/2} -${PI/2}" xyz="0 0 -${finger_length/2}"/>
@@ -161,5 +216,5 @@
         <axis xyz="0 1 0"/>
         <origin rpy="0 0 0" xyz="${-gripper_joint_x} ${gripper_joint_y} ${gripper_joint_z}"/>
-        <limit lower="0" upper="${PI/2}" effort="${effort}" velocity="${velocity}"/>
+        <limit lower="${-PI/9}" upper="${PI/2}" effort="${effort}" velocity="${velocity}"/>
     </joint>
     <joint name="gripper_joint_2" type="revolute">
@@ -169,5 +224,5 @@
         <origin rpy="0 0 0" xyz="${gripper_joint_x} ${gripper_joint_y} ${gripper_joint_z}"/>
         <mimic joint="gripper_joint_1" multiplier="-1"/>
-        <limit lower="0" upper="${PI/2}" effort="${effort}" velocity="${velocity}"/>
+        <limit lower="${-PI/9}" upper="${PI/2}" effort="${effort}" velocity="${velocity}"/>
     </joint>
 </robot>

Commit message: change model is supposed to be working (need to set an srdf)

File: theseus_description/urdf/manipulator.urdf.xacro (robot description, xacro)
@@ -64,9 +64,31 @@
         <parent link="base_link"/>
         <child link="arm_link_1"/>
+        <axis xyz="0 0 1"/>
+        <origin rpy="0 0 0" xyz="0 0 0.06"/>
+        <limit lower="0" upper="${3*PI/2}" effort="${effort}" velocity="${velocity}"/>
+    </joint>
+    <link name="arm_link_2">
+        <xacro:default_inertial mass="1.0"/>
+        <visual>
+            <origin rpy="0 0 0" xyz="0 0 ${link1_length/2}"/>
+            <geometry>
+                <cylinder radius="0.05" length="${link1_length}"/>
+            </geometry>
+        </visual>
+        <collision>
+            <origin rpy="0 0 0" xyz="0 0 ${link1_length/2}"/>
+            <geometry>
+                <cylinder radius="0.05" length="${link1_length}"/>
+            </geometry>
+        </collision>
+    </link>
+    <joint name="arm_joint_2" type="revolute">
+        <parent link="base_link"/>
+        <child link="arm_link_1"/>
         <axis xyz="0 1 0"/>
         <origin rpy="0 0 0" xyz="0 0 0.06"/>
-        <limit lower="-${3*PI/4}" upper="${3*PI/4}" effort="${effort}" velocity="${velocity}"/>
+        <limit lower="0" upper="${3*PI/2}" effort="${effort}" velocity="${velocity}"/>
     </joint>
-     <link name="arm_link_2">
+     <link name="arm_link_3">
         <xacro:default_inertial mass="1.0"/>
         <visual>
@@ -83,5 +105,5 @@
         </collision>
     </link>
-    <joint name="arm_joint_2" type="revolute">
+    <joint name="arm_joint_3" type="revolute">
         <parent link="arm_link_1"/>
         <child link="arm_link_2"/>

File: theseus_description/urdf/manipulator_ros2_control.xacro (robot description, xacro)
@@ -29,11 +29,11 @@
             <hardware>
                 <plugin>theseus_controller/TheseusInterface</plugin>
-                <param name="port">/dev/ttyACM0</param>
+                <param name="port">/dev/ttyUSB0</param>
             </hardware>
         </xacro:unless>
         <joint name="arm_joint_1">
             <command_interface name="position">
-            <param name="min">-${3*PI/4}</param>
-            <param name="max">${3*PI/4}</param>
+            <param name="min">0</param>
+            <param name="max">${3*PI/2}</param>
             </command_interface>
             <state_interface name="position"/>
@@ -41,6 +41,13 @@
         <joint name="arm_joint_2">
             <command_interface name="position">
-            <param name="min">-${3*PI/4}</param>
-            <param name="max">${3*PI/4}</param>
+            <param name="min">0</param>
+            <param name="max">${3*PI/2}</param>
+            </command_interface>
+            <state_interface name="position"/>
+        </joint>
+        <joint name="arm_joint_3">
+            <command_interface name="position">
+            <param name="min">0</param>
+            <param name="max">${3*PI/2}</param>
             </command_interface>
             <state_interface name="position"/>

Commit message: erro no move_group para urdf manipulator, need to change moveit_controllers in launch according to urdf

File: theseus_description/urdf/manipulator.urdf.xacro (robot description, xacro)
@@ -1,4 +1,4 @@
 <?xml version="1.0"?>
-<robot xmlns:xacro="http://www.ros.org/wiki/xacro" name="utbots_manipulator">
+<robot xmlns:xacro="http://www.ros.org/wiki/xacro" name="manipulator">
     <!-- TODO Adjust all links, joints, visuals, collision and inertias for theseus -->
     <xacro:arg name="is_sim" default="false" />
@@ -49,13 +49,13 @@
         <xacro:default_inertial mass="1.0"/>
         <visual>
-            <origin rpy="0 0 0" xyz="0 0 ${link1_length/2}"/>
+            <origin rpy="0 0 0" xyz="0 0 0"/>
             <geometry>
-                <cylinder radius="0.05" length="${link1_length}"/>
+                <cylinder radius="0.05" length="0"/>
             </geometry>
         </visual>
         <collision>
-            <origin rpy="0 0 0" xyz="0 0 ${link1_length/2}"/>
+            <origin rpy="0 0 0" xyz="0 0 0"/>
             <geometry>
-                <cylinder radius="0.05" length="${link1_length}"/>
+                <cylinder radius="0.05" length="0"/>
             </geometry>
         </collision>
@@ -65,6 +65,6 @@
         <child link="arm_link_1"/>
         <axis xyz="0 0 1"/>
-        <origin rpy="0 0 0" xyz="0 0 0.06"/>
-        <limit lower="0" upper="${3*PI/2}" effort="${effort}" velocity="${velocity}"/>
+        <origin rpy="0 0 0" xyz="0 0 0"/>
+        <limit lower="-${3*PI/4}" upper="${3*PI/4}" effort="${effort}" velocity="${velocity}"/>
     </joint>
     <link name="arm_link_2">
@@ -84,9 +84,9 @@
     </link>
     <joint name="arm_joint_2" type="revolute">
-        <parent link="base_link"/>
-        <child link="arm_link_1"/>
+        <parent link="arm_link_1"/>
+        <child link="arm_link_2"/>
         <axis xyz="0 1 0"/>
         <origin rpy="0 0 0" xyz="0 0 0.06"/>
-        <limit lower="0" upper="${3*PI/2}" effort="${effort}" velocity="${velocity}"/>
+        <limit lower="-${3*PI/4}" upper="${3*PI/4}" effort="${effort}" velocity="${velocity}"/>
     </joint>
      <link name="arm_link_3">
@@ -106,6 +106,6 @@
     </link>
     <joint name="arm_joint_3" type="revolute">
-        <parent link="arm_link_1"/>
-        <child link="arm_link_2"/>
+        <parent link="arm_link_2"/>
+        <child link="arm_link_3"/>
         <axis xyz="0 1 0"/>
         <origin rpy="0 0 0" xyz="0 0 ${link1_length}"/>
@@ -128,5 +128,5 @@
     </link>
     <joint name="arm_to_claw_joint" type="fixed">
-        <parent link="arm_link_2"/>
+        <parent link="arm_link_3"/>
         <child link="claw_link"/>
         <origin rpy="0 0 0" xyz="0 0 ${link2_length}"/>

File: theseus_description/urdf/manipulator_ros2_control.xacro (robot description, xacro)
@@ -1,4 +1,4 @@
 <?xml version="1.0"?>
-<robot xmlns:xacro="http://www.ros.org/wiki/xacro" name="utbots_manipulator">
+<robot xmlns:xacro="http://www.ros.org/wiki/xacro" name="manipulator">
     <ros2_control name="ManipulatorSystem" type="system">
         <xacro:property name="PI" value="3.14159265358979323846"/>
@@ -34,6 +34,6 @@
         <joint name="arm_joint_1">
             <command_interface name="position">
-            <param name="min">0</param>
-            <param name="max">${3*PI/2}</param>
+            <param name="min">${-3*PI/4}</param>
+            <param name="max">${3*PI/4}</param>
             </command_interface>
             <state_interface name="position"/>
@@ -41,6 +41,6 @@
         <joint name="arm_joint_2">
             <command_interface name="position">
-            <param name="min">0</param>
-            <param name="max">${3*PI/2}</param>
+            <param name="min">${-3*PI/4}</param>
+            <param name="max">${3*PI/4}</param>
             </command_interface>
             <state_interface name="position"/>
@@ -48,6 +48,6 @@
         <joint name="arm_joint_3">
             <command_interface name="position">
-            <param name="min">0</param>
-            <param name="max">${3*PI/2}</param>
+            <param name="min">${-3*PI/4}</param>
+            <param name="max">${3*PI/4}</param>
             </command_interface>
             <state_interface name="position"/>

Commit message: inverse kinematics working both simulaion and real with different models, bringup launch ok

File: theseus_description/urdf/manipulator.urdf.xacro (robot description, xacro)
@@ -5,5 +5,5 @@
     <xacro:arg name="is_ignition" default="true" />
     <!-- Include Gazebo Parameters (only relevant for sim) -->
-    <xacro:include filename="$(find theseus_description)/urdf/theseus_gazebo.xacro"/>
+    <xacro:include filename="$(find theseus_description)/urdf/manipulator_gazebo.xacro"/>
     <!-- Include ros2_control plugins -->
     <xacro:include filename="$(find theseus_description)/urdf/manipulator_ros2_control.xacro"/>
@@ -49,13 +49,13 @@
         <xacro:default_inertial mass="1.0"/>
         <visual>
-            <origin rpy="0 0 0" xyz="0 0 0"/>
+            <origin rpy="0 0 0" xyz="0 0 0.03"/>
             <geometry>
-                <cylinder radius="0.05" length="0"/>
+                <cylinder radius="0.05" length="0.06"/>
             </geometry>
         </visual>
         <collision>
-            <origin rpy="0 0 0" xyz="0 0 0"/>
+            <origin rpy="0 0 0" xyz="0 0 0.03"/>
             <geometry>
-                <cylinder radius="0.05" length="0"/>
+                <cylinder radius="0.05" length="0.06"/>
             </geometry>
         </collision>
@@ -65,5 +65,5 @@
         <child link="arm_link_1"/>
         <axis xyz="0 0 1"/>
-        <origin rpy="0 0 0" xyz="0 0 0"/>
+        <origin rpy="0 0 0" xyz="0 0 0.06"/>
         <limit lower="-${3*PI/4}" upper="${3*PI/4}" effort="${effort}" velocity="${velocity}"/>
     </joint>

File: theseus_description/urdf/theseus.urdf.xacro (robot description, xacro)
@@ -20,5 +20,5 @@
     <xacro:property name="effort" value="10.0"/>
     <xacro:property name="velocity" value="5.0"/>
-    <!-- Mesh scale -->
+    <!-- Mesh rendering properties -->
     <xacro:property name="mesh_scale" value="0.003 0.003 0.003"/>
     <material name="default_red">

Commit message: end effector ok in theseus model

File: theseus_description/urdf/manipulator.urdf.xacro (robot description, xacro)
@@ -132,4 +132,10 @@
         <origin rpy="0 0 0" xyz="0 0 ${link2_length}"/>
     </joint>
+    <link name="gripper_center"/>
+    <joint name="gripper_center_joint">
+        <parent link="claw_link"/>
+        <child link="gripper_center"/>
+        <origin rpy="0 0 0" xyz="0 0 ${-finger_length/2}"/>
+    </joint>
     <link name="gripper_right">
         <xacro:default_inertial mass="1.0"/>

File: theseus_description/urdf/theseus.urdf.xacro (robot description, xacro)
@@ -194,4 +194,10 @@
         </collision>
     </link>
+    <link name="gripper_center"/>
+    <joint name="gripper_center_joint" type="fixed">
+        <parent link="gripper_link"/>
+        <child link="gripper_center"/>
+        <origin rpy="0 ${PI/2} -${PI/2}" xyz="-0 0 -${3*finger_length}"/>
+    </joint>
     <joint name="gripper_joint" type="revolute">
         <parent link="arm_link_4"/>
