Commit message: updated urdf with variables

File: theseus_description/urdf/manipulator.urdf.xacro (robot description, xacro)
@@ -13,8 +13,35 @@
     <xacro:property name="velocity" value="5.0"/>
     <!-- Link -->
+    <xacro:property name="link2_length" value="0.235"/>
+    <xacro:property name="step_reductor_height" value="0.025"/>
+    <xacro:property name="finger_length" value="0.15"/>
+    <!-- Arm Base Link  -->
+    <xacro:property name="base_cilinder_height" value="0.025"/>
+    <xacro:property name="base_cilinder_radius" value="0.08"/>
+    <xacro:property name="base_servo_distance_from_center" value="0.08"/>
+    <xacro:property name="joint_1_lower_limit" value="0"/>
+    <xacro:property name="joint_1_upper_limit" value="${2*PI}"/>
+    <!-- Arm Link 1 -->
+    <xacro:property name="servo_motor_1_width" value="0.05"/>
+    <xacro:property name="servo_motor_1_depth" value="0.03"/>
+    <xacro:property name="servo_motor_1_height" value="0.06"/>
+    <xacro:property name="servo_motor_1_angle" value="${PI/4}"/>
+    <xacro:property name="servo_motor_1_offset_angle" value="-${3*PI/4}"/>
+    <xacro:property name="servo_hinge_1_width" value="0.065"/>
+    <xacro:property name="servo_hinge_1_depth" value="0.03"/>
+    <xacro:property name="servo_hinge_1_height" value="0.035"/>
+    <xacro:property name="joint_2_lower_limit" value="${PI/4}"/>
+    <xacro:property name="joint_2_upper_limit" value="${3*PI/2}"/>
     <xacro:property name="link1_length" value="0.275"/>
-    <xacro:property name="link2_length" value="0.235"/>
-    <!-- <xacro:property name="" -->
-    <xacro:property name="finger_length" value="0.15"/>
+    <!-- Arm Link 2 -->
+    <xacro:property name="servo_motor_2_width" value="0.05"/>
+    <xacro:property name="servo_motor_2_depth" value="0.03"/>
+    <xacro:property name="servo_motor_2_height" value="0.06"/>
+    <xacro:property name="servo_motor_2_offset_angle" value="-${3*PI/4}"/>
+    <xacro:property name="servo_hinge_2_width" value="0.065"/>
+    <xacro:property name="servo_hinge_2_depth" value="0.03"/>
+    <xacro:property name="servo_hinge_2_height" value="0.035"/>
+    <xacro:property name="joint_3_lower_limit" value="${3*PI/4}"/>
+    <xacro:property name="joint_3_upper_limit" value="${3*PI/2}"/>
     <!-- Macros -->
     <xacro:macro name="default_inertial" params="mass">
@@ -31,13 +58,13 @@
         <xacro:default_inertial mass="1.0"/>
         <visual>
-            <origin rpy="0 0 0" xyz="0 0 0.025"/>
-            <geometry>
-                <cylinder radius="0.08" length="0.025"/>
-            </geometry>
-        </visual>
-        <collision>
-            <origin rpy="0 0 0" xyz="0 0 0.025"/>
-            <geometry>
-                <cylinder radius="0.08" length="0.025"/>
+            <origin rpy="0 0 0" xyz="0 0 ${base_cilinder_height}"/>
+            <geometry>
+                <cylinder radius="${base_cilinder_radius}" length="${base_cilinder_height}"/>
+            </geometry>
+        </visual>
+        <collision>
+            <origin rpy="0 0 0" xyz="0 0 ${base_cilinder_height}"/>
+            <geometry>
+                <cylinder radius="${base_cilinder_radius}" length="${base_cilinder_height}"/>
             </geometry>
         </collision>
@@ -47,19 +74,19 @@
         <child link="base_arm_link"/>
         <axis xyz="0 0 1"/>
-        <origin rpy="0 0 0.055" xyz="0 0 0.025"/>
-        <limit lower="0" upper="${2*PI}" effort="${effort}" velocity="${velocity}"/>
+        <origin rpy="0 0 0" xyz="0 0 ${base_cilinder_height}"/>
+        <limit lower="${joint_1_lower_limit}" upper="${joint_1_upper_limit}" effort="${effort}" velocity="${velocity}"/>
     </joint>
     <link name="motor_link_1">
         <xacro:default_inertial mass="1.0"/>
         <visual>
-            <origin rpy="0 0 0" xyz="0 0 0.03"/>
-            <geometry>
-                <box size="0.05 0.03 0.06"/>
-            </geometry>
-        </visual>
-        <collision>
-            <origin rpy="0 0 0" xyz="0 0 0.03"/>
-            <geometry>
-                <box size="0.05 0.03 0.06"/>
+            <origin rpy="0 0 0" xyz="0 0 ${servo_motor_1_depth}"/>
+            <geometry>
+                <box size="${servo_motor_1_width} ${servo_motor_1_depth} ${servo_motor_1_height}"/>
+            </geometry>
+        </visual>
+        <collision>
+            <origin rpy="0 0 0" xyz="0 0 ${servo_motor_1_depth}"/>
+            <geometry>
+                <box size="${servo_motor_1_width} ${servo_motor_1_depth} ${servo_motor_1_height}"/>
             </geometry>
         </collision>
@@ -68,19 +95,20 @@
         <parent link="base_arm_link"/>
         <child link="motor_link_1"/>
-        <origin rpy="${PI/4} 0 0" xyz="0 -0.04 0.03"/>
+        <origin rpy="${servo_motor_1_angle} 0 0" xyz="0 -${servo_motor_1_depth} ${servo_motor_1_width}"/>
     </joint>
     <link name="hinge_link_1">
         <xacro:default_inertial mass="1.0"/>
         <visual>
-            <origin rpy="0 0 0" xyz="0 0 0.0175"/>
-            <geometry>
-                <box size="0.065 0.03 0.035"/>
+            <origin rpy="0 0 0" xyz="0 0 ${servo_hinge_1_height/2}"/>
+            <geometry>
+                <box size="${servo_hinge_1_width} ${servo_hinge_1_depth} ${servo_hinge_1_height}"/>
             </geometry>
         </visual>
         <!-- <collision>
-            <origin rpy="0 0 0" xyz="0 0 0.0175"/>
-            <geometry>
-                <box size="0.065 0.03 0.035"/>
-            </geometry>
+            <origin rpy="0 0 0" xyz="0 0 ${servo_hinge_1_height/2}"/>
+            <geometry>
+                <box size="${servo_hinge_1_width} ${servo_hinge_1_depth} ${servo_hinge_1_height}"/>
+            </geometry>
+        </visual>
         </collision> -->
     </link>
@@ -88,9 +116,9 @@
         <parent link="motor_link_1"/>
         <child link="hinge_link_1"/>
-        <origin rpy="-${3*PI/4} 0 0" xyz="0 0 0.06"/>
-        <axis xyz="1 0 0"/>
-        <limit lower="${PI/4}" upper="${3*PI/2}" effort="${effort}" velocity="${velocity}"/>
-    </joint>
-    <link name="arm_link_2">
+        <origin rpy="${servo_motor_1_offset_angle} 0 0" xyz="0 0 ${servo_motor_1_height}"/>
+        <axis xyz="1 0 0"/>
+        <limit lower="${joint_2_lower_limit}" upper="${joint_2_upper_limit}" effort="${effort}" velocity="${velocity}"/>
+    </joint>
+    <link name="arm_link_1">
         <xacro:default_inertial mass="1.0"/>
         <visual>
@@ -109,24 +137,24 @@
     <joint name="arm_joint_2" type="fixed">
         <parent link="hinge_link_1"/>
-        <child link="arm_link_2"/>
-        <origin rpy="0 0 0" xyz="0 0 0.035"/>
+        <child link="arm_link_1"/>
+        <origin rpy="0 0 0" xyz="0 0 ${servo_hinge_1_height}"/>
     </joint>
     <link name="motor_link_2">
         <xacro:default_inertial mass="1.0"/>
-        <visual>
-            <origin rpy="0 0 0" xyz="0 0 0.03"/>
-            <geometry>
-                <box size="0.05 0.03 0.06"/>
-            </geometry>
-        </visual>
-        <collision>
-            <origin rpy="0 0 0" xyz="0 0 0.03"/>
-            <geometry>
-                <box size="0.05 0.03 0.06"/>
+                <visual>
+            <origin rpy="0 0 0" xyz="0 0 ${servo_motor_2_depth}"/>
+            <geometry>
+                <box size="${servo_motor_2_width} ${servo_motor_2_depth} ${servo_motor_2_height}"/>
+            </geometry>
+        </visual>
+        <collision>
+            <origin rpy="0 0 0" xyz="0 0 ${servo_motor_2_depth}"/>
+            <geometry>
+                <box size="${servo_motor_2_width} ${servo_motor_2_depth} ${servo_motor_2_height}"/>
             </geometry>
         </collision>
     </link>
     <joint name="motor_joint_2" type="fixed">
-        <parent link="arm_link_2"/>
+        <parent link="arm_link_1"/>
         <child link="motor_link_2"/>
         <origin rpy="0 0 0" xyz="0 0 ${link2_length}"/>
@@ -135,13 +163,13 @@
         <xacro:default_inertial mass="1.0"/>
         <visual>
-            <origin rpy="0 0 0" xyz="0 0 0.0175"/>
-            <geometry>
-                <box size="0.065 0.03 0.035"/>
+            <origin rpy="0 0 0" xyz="0 0 ${servo_hinge_2_height/2}"/>
+            <geometry>
+                <box size="${servo_hinge_2_width} ${servo_hinge_2_depth} ${servo_hinge_2_height}"/>
             </geometry>
         </visual>
         <!-- <collision>
-            <origin rpy="0 0 0" xyz="0 0 0.0175"/>
-            <geometry>
-                <box size="0.065 0.03 0.035"/>
+            <origin rpy="0 0 0" xyz="0 0 ${servo_hinge_2_height/2}"/>
+            <geometry>
+                <box size="${servo_hinge_2_width} ${servo_hinge_2_depth} ${servo_hinge_2_height}"/>
             </geometry>
         </collision> -->
@@ -150,9 +178,9 @@
         <parent link="motor_link_2"/>
         <child link="hinge_link_2"/>
-        <origin rpy="-${3*PI/4} 0 0" xyz="0 0 0.06"/>
-        <axis xyz="1 0 0"/>
-        <limit lower="${3*PI/4}" upper="${3*PI/2}" effort="${effort}" velocity="${velocity}"/>
-    </joint>
-     <link name="arm_link_3">
+        <origin rpy="${servo_motor_2_offset_angle} 0 0" xyz="0 0 ${servo_motor_2_height}"/>
+        <axis xyz="1 0 0"/>
+        <limit lower="${joint_2_lower_limit}" upper="${joint_2_upper_limit}" effort="${effort}" velocity="${velocity}"/>
+    </joint>
+     <link name="arm_link_2">
         <xacro:default_inertial mass="1.0"/>
         <visual>
@@ -171,6 +199,6 @@
     <joint name="arm_joint_3" type="fixed">
         <parent link="hinge_link_2"/>
-        <child link="arm_link_3"/>
-        <origin rpy="0 0 0" xyz="0 0 0.035"/>
+        <child link="arm_link_2"/>
+        <origin rpy="0 0 0" xyz="0 0 ${servo_hinge_2_height}"/>
     </joint>
     <link name="claw_link">
@@ -190,5 +218,5 @@
     </link>
     <joint name="arm_to_claw_joint" type="fixed">
-        <parent link="arm_link_3"/>
+        <parent link="arm_link_2"/>
         <child link="claw_link"/>
         <origin rpy="0 0 0" xyz="0 0 ${link2_length}"/>

File: theseus_description/urdf/manipulator_ros2_control.xacro (robot description, xacro)
@@ -34,20 +34,20 @@
         <joint name="arm_joint_1">
             <command_interface name="position">
-            <param name="min">${-3*PI/4}</param>
-            <param name="max">${3*PI/4}</param>
+            <param name="min">0</param>
+            <param name="max">${2*PI}</param>
             </command_interface>
             <state_interface name="position"/>
         </joint>
-        <joint name="arm_joint_2">
+        <joint name="hinge_joint_1">
             <command_interface name="position">
-            <param name="min">${-3*PI/4}</param>
-            <param name="max">${3*PI/4}</param>
+            <param name="min">${PI/4}</param>
+            <param name="max">${3*PI/2}</param>
             </command_interface>
             <state_interface name="position"/>
         </joint>
-        <joint name="arm_joint_3">
+        <joint name="hinge_joint_2">
             <command_interface name="position">
-            <param name="min">${-3*PI/4}</param>
-            <param name="max">${3*PI/4}</param>
+            <param name="min">${3*PI/4}</param>
+            <param name="max">${3*PI/2}</param>
             </command_interface>
             <state_interface name="position"/>

Commit message: REAL MANIPULATOR CONTROL WORKING WITH KINEMATICS

File: theseus_description/urdf/manipulator.urdf.xacro (robot description, xacro)
@@ -73,5 +73,5 @@
         <parent link="world"/>
         <child link="base_arm_link"/>
-        <axis xyz="0 0 1"/>
+        <axis xyz="0 0 -1"/>
         <origin rpy="0 0 0" xyz="0 0 ${base_cilinder_height}"/>
         <limit lower="${joint_1_lower_limit}" upper="${joint_1_upper_limit}" effort="${effort}" velocity="${velocity}"/>
@@ -105,11 +105,10 @@
             </geometry>
         </visual>
-        <!-- <collision>
-            <origin rpy="0 0 0" xyz="0 0 ${servo_hinge_1_height/2}"/>
-            <geometry>
-                <box size="${servo_hinge_1_width} ${servo_hinge_1_depth} ${servo_hinge_1_height}"/>
-            </geometry>
-        </visual>
-        </collision> -->
+        <collision>
+            <origin rpy="0 0 0" xyz="0 0 ${servo_hinge_1_height/2+servo_hinge_1_height/3}"/>
+            <geometry>
+                <box size="${servo_hinge_1_width} ${servo_hinge_1_depth} ${servo_hinge_2_height/3}"/>
+            </geometry>
+        </collision>
     </link>
     <joint name="hinge_joint_1" type="revolute">
@@ -158,5 +157,5 @@
         <parent link="arm_link_1"/>
         <child link="motor_link_2"/>
-        <origin rpy="0 0 0" xyz="0 0 ${link2_length}"/>
+        <origin rpy="0 0 0" xyz="0 0 ${link2_length+servo_motor_2_height/2}"/>
     </joint>
     <link name="hinge_link_2">
@@ -168,10 +167,10 @@
             </geometry>
         </visual>
-        <!-- <collision>
-            <origin rpy="0 0 0" xyz="0 0 ${servo_hinge_2_height/2}"/>
-            <geometry>
-                <box size="${servo_hinge_2_width} ${servo_hinge_2_depth} ${servo_hinge_2_height}"/>
-            </geometry>
-        </collision> -->
+        <collision>
+            <origin rpy="0 0 0" xyz="0 0 ${servo_hinge_2_height/2+servo_hinge_2_height/3}"/>
+            <geometry>
+                <box size="${servo_hinge_2_width} ${servo_hinge_2_depth} ${servo_hinge_2_height/3}"/>
+            </geometry>
+        </collision>
     </link>
     <joint name="hinge_joint_2" type="revolute">
@@ -180,5 +179,5 @@
         <origin rpy="${servo_motor_2_offset_angle} 0 0" xyz="0 0 ${servo_motor_2_height}"/>
         <axis xyz="1 0 0"/>
-        <limit lower="${joint_2_lower_limit}" upper="${joint_2_upper_limit}" effort="${effort}" velocity="${velocity}"/>
+        <limit lower="${joint_3_lower_limit}" upper="${joint_3_upper_limit}" effort="${effort}" velocity="${velocity}"/>
     </joint>
      <link name="arm_link_2">

Commit message: manipulator urdf with real gripper

File: theseus_description/urdf/manipulator.urdf.xacro (robot description, xacro)
@@ -8,4 +8,6 @@
     <!-- Include ros2_control plugins -->
     <xacro:include filename="$(find theseus_description)/urdf/manipulator_ros2_control.xacro"/>
+    <!-- Mesh scale -->
+    <xacro:property name="mesh_scale" value="0.001 0.001 0.001"/>
     <!-- Useful XACRO variables -->
     <xacro:property name="PI" value="3.14159265358979323846"/>
@@ -204,13 +206,13 @@
         <xacro:default_inertial mass="1.0"/>
         <visual>
+            <origin rpy="0 ${PI/2} 0" xyz="-0.09 -0.095 -0.12"/>
+            <geometry>
+                <mesh filename="package://theseus_description/meshes/pulso-garra.stl" scale="${mesh_scale}"/>
+            </geometry>
+        </visual>
+        <collision>
             <origin rpy="0 0 0" xyz="0 0 0.01"/>
             <geometry>
-                <cylinder radius="0.04" length="0.02"/>
-            </geometry>
-        </visual>
-        <collision>
-            <origin rpy="0 0 0" xyz="0 0 0.01"/>
-            <geometry>
-                <cylinder radius="0.04" length="0.02"/>
+                <mesh filename="package://theseus_description/meshes/pulso-garra.stl" scale="${mesh_scale}"/>
             </geometry>
         </collision>
@@ -230,13 +232,13 @@
         <xacro:default_inertial mass="1.0"/>
         <visual>
-            <origin rpy="0 0 -${PI/2}" xyz="0 -0.02 ${finger_length/2}"/>
-            <geometry>
-                <cylinder radius="0.02" length="${finger_length}"/>
-            </geometry>
-        </visual>
-        <collision>
-            <origin rpy="0 0 -${PI/2}" xyz="0 -0.02 ${finger_length/2}"/>
-            <geometry>
-                <cylinder radius="0.02" length="${finger_length}"/>
+            <origin rpy="0 0 0" xyz="-0.0825 -0.08 0.0975"/>
+            <geometry>
+                <mesh filename="package://theseus_description/meshes/palma-garra.stl" scale="${mesh_scale}"/>
+            </geometry>
+        </visual>
+        <collision>
+            <origin rpy="0 0 0" xyz="-0.0825 -0.08 0.0975"/>
+            <geometry>
+                <mesh filename="package://theseus_description/meshes/palma-garra.stl" scale="${mesh_scale}"/>
             </geometry>
         </collision>
@@ -245,13 +247,13 @@
         <xacro:default_inertial mass="1.0"/>
         <visual>
-            <origin rpy="0 0 -${PI/2}" xyz="0 0.02 ${finger_length/2}"/>
-            <geometry>
-                <cylinder radius="0.02" length="${finger_length}"/>
-            </geometry>
-        </visual>
-        <collision>
-            <origin rpy="0 0 -${PI/2}" xyz="0 -0.02 ${finger_length/2}"/>
-            <geometry>
-                <cylinder radius="0.02" length="${finger_length}"/>
+            <origin rpy="0 0 -${PI}" xyz="0.0825 0.08 0.0975"/>
+            <geometry>
+                <mesh filename="package://theseus_description/meshes/palma-garra.stl" scale="${mesh_scale}"/>
+            </geometry>
+        </visual>
+        <collision>
+            <origin rpy="0 0 -${PI}" xyz="0.0825 0.08 0.0975"/>
+            <geometry>
+                <mesh filename="package://theseus_description/meshes/palma-garra.stl" scale="${mesh_scale}"/>
             </geometry>
         </collision>
@@ -260,6 +262,6 @@
         <parent link="claw_link"/>
         <child link="gripper_right"/>
-        <axis xyz="1 0 0"/>
-        <origin rpy="0 0 0" xyz="0 0 0"/>
+        <axis xyz="0 1 0"/>
+        <origin rpy="0 0 0" xyz="0.015 0 0.05"/>
         <limit lower="0" upper="${PI/2}" effort="${effort}" velocity="${velocity}"/>
     </joint>
@@ -267,6 +269,6 @@
         <parent link="claw_link"/>
         <child link="gripper_left"/>
-        <axis xyz="1 0 0"/>
-        <origin rpy="0 0 0" xyz="0 0 0"/>
+        <axis xyz="0 1 0"/>
+        <origin rpy="0 0 0" xyz="-0.015 0 0.05"/>
         <mimic joint="gripper_joint_1" multiplier="-1"/>
         <limit lower="0" upper="${PI/2}" effort="${effort}" velocity="${velocity}"/>

Commit message: gripper controller adjustments

File: theseus_description/urdf/manipulator.urdf.xacro (robot description, xacro)
@@ -227,5 +227,5 @@
         <parent link="claw_link"/>
         <child link="gripper_center"/>
-        <origin rpy="0 0 0" xyz="0 0 ${-finger_length/2}"/>
+        <origin rpy="0 0 0" xyz="0 0 0.07"/>
     </joint>
     <link name="gripper_right">

Commit message: attempts at inverse kinematics test for 30, 90 and 225 angles

File: theseus_description/urdf/manipulator.urdf.xacro (robot description, xacro)
@@ -159,5 +159,5 @@
         <parent link="arm_link_1"/>
         <child link="motor_link_2"/>
-        <origin rpy="0 0 0" xyz="0 0 ${link2_length+servo_motor_2_height/2}"/>
+        <origin rpy="0 0 0" xyz="0 0 ${link1_length+servo_motor_2_height/2}"/>
     </joint>
     <link name="hinge_link_2">

Commit message: configs seem to be ok

File: theseus_description/urdf/manipulator.urdf.xacro (robot description, xacro)
@@ -159,5 +159,5 @@
         <parent link="arm_link_1"/>
         <child link="motor_link_2"/>
-        <origin rpy="0 0 0" xyz="0 0 ${link1_length+servo_motor_2_height/2}"/>
+        <origin rpy="0 0 0" xyz="0 0 ${link1_length}"/>
     </joint>
     <link name="hinge_link_2">

Commit message: adjustments in cbr

File: theseus_description/urdf/manipulator.urdf.xacro (robot description, xacro)
@@ -75,5 +75,5 @@
         <parent link="world"/>
         <child link="base_arm_link"/>
-        <axis xyz="0 0 -1"/>
+        <axis xyz="0 0 1"/>
         <origin rpy="0 0 0" xyz="0 0 ${base_cilinder_height}"/>
         <limit lower="${joint_1_lower_limit}" upper="${joint_1_upper_limit}" effort="${effort}" velocity="${velocity}"/>
