Commit message: working theseus simulation, but action server still having goals rejected, manipulator model simulation not working

File: theseus_description/urdf/manipulator.urdf.xacro (robot description, xacro)
@@ -5,5 +5,5 @@
     <xacro:arg name="is_ignition" default="true" />
     <!-- Include Gazebo Parameters (only relevant for sim) -->
-    <!-- <xacro:include filename="$(find theseus_description)/urdf/manipulator_gazebo.xacro"/> -->
+    <xacro:include filename="$(find theseus_description)/urdf/manipulator_gazebo.xacro"/>
     <!-- Include ros2_control plugins -->
     <xacro:include filename="$(find theseus_description)/urdf/manipulator_ros2_control.xacro"/>
@@ -75,5 +75,5 @@
         <parent link="world"/>
         <child link="base_arm_link"/>
-        <axis xyz="0 0 1"/>
+        <axis xyz="0 0 -1"/>
         <origin rpy="0 0 0" xyz="0 0 ${base_cilinder_height}"/>
         <limit lower="${joint_1_lower_limit}" upper="${joint_1_upper_limit}" effort="${effort}" velocity="${velocity}"/>
@@ -269,5 +269,5 @@
         <parent link="claw_link"/>
         <child link="gripper_left"/>
-        <axis xyz="0 1 0"/>
+        <!-- <axis xyz="0 1 0"/> -->
         <origin rpy="0 0 0" xyz="-0.015 0 0.05"/>
         <mimic joint="gripper_joint_1" multiplier="-1"/>

File: theseus_description/urdf/manipulator_ros2_control.xacro (robot description, xacro)
@@ -3,4 +3,5 @@
     <ros2_control name="ManipulatorSystem" type="system">
         <xacro:property name="PI" value="3.14159265358979323846"/>
+        <xacro:property name="initial_positions" value="$(find theseus_moveit)/config/manipulator/initial_positions.yaml"/>
         <!-- ros2_control Gazebo only -->
         <xacro:if value="$(arg is_sim)">
@@ -15,13 +16,4 @@
                 </hardware>
             </xacro:unless>
-            <joint name="gripper_joint_2">
-                <param name="mimic">gripper_joint_1</param>
-                <param name="multiplier">-1</param>
-                <command_interface name="position">
-                <param name="min">0</param>
-                <param name="max">${PI/2}</param>
-                </command_interface>
-                <state_interface name="position"/>
-            </joint>
         </xacro:if>
         <!-- ros2_control real manipulator only -->
@@ -43,4 +35,5 @@
             <param name="min">${PI/4}</param>
             <param name="max">${3*PI/2}</param>
+            <param name="initial_position">0.785398</param>
             </command_interface>
             <state_interface name="position"/>
@@ -50,4 +43,5 @@
             <param name="min">${3*PI/4}</param>
             <param name="max">${3*PI/2}</param>
+            <param name="initial_position">4.71238</param>
             </command_interface>
             <state_interface name="position"/>
@@ -57,4 +51,5 @@
             <param name="min">0</param>
             <param name="max">${PI/2}</param>
+            <param name="initial_position">0</param>
             </command_interface>
             <state_interface name="position"/>

File: theseus_description/urdf/theseus_ros2_control.xacro (robot description, xacro)
@@ -3,5 +3,5 @@
     <ros2_control name="ManipulatorSystem" type="system">
         <xacro:property name="PI" value="3.14159265358979323846"/>
-        <xacro:property name="initial_positions" value="$(find theseus_moveit)/config/initial_positions.yaml"/>
+        <xacro:property name="initial_positions" value="$(find theseus_moveit)/config/theseus/initial_positions.yaml"/>
         <!-- ros2_control Gazebo only -->
         <xacro:if value="$(arg is_sim)">
