Commit message: half of controllers, urdf with gripper

File: theseus_description/urdf/theseus.urdf.xacro (robot description, xacro)
@@ -4,4 +4,7 @@
     <xacro:property name="effort" value="10.0"/>
     <xacro:property name="velocity" value="5.0"/>
+    <xacro:property name="link1_length" value="0.34"/>
+    <xacro:property name="link2_length" value="0.27"/>
+    <xacro:property name="finger_length" value="0.15"/>
     <link name="world"/>
     <link name="base_link">
@@ -20,7 +23,7 @@
     <link name="arm_link_1">
         <visual>
-            <origin rpy="0 0 0" xyz="0 0 0.17"/>
+            <origin rpy="0 0 0" xyz="0 0 ${link1_length/2}"/>
             <geometry>
-                <cylinder radius="0.05" length="0.34"/>
+                <cylinder radius="0.05" length="${link1_length}"/>
             </geometry>
         </visual>
@@ -31,11 +34,11 @@
         <axis xyz="0 1 0"/>
         <origin rpy="0 0 0" xyz="0 0 0.06"/>
-        <limit lower="-${PI/2}" upper="${PI/2}" effort="${effort}" velocity="${velocity}"/>
+        <limit lower="-${3*PI/4}" upper="${3*PI/4}" effort="${effort}" velocity="${velocity}"/>
     </joint>
      <link name="arm_link_2">
         <visual>
-            <origin rpy="0 0 0" xyz="0 0 0.135"/>
+            <origin rpy="0 0 0" xyz="0 0 ${link2_length/2}"/>
             <geometry>
-                <cylinder radius="0.05" length="0.27"/>
+                <cylinder radius="0.05" length="${link2_length}"/>
             </geometry>
         </visual>
@@ -45,7 +48,71 @@
         <child link="arm_link_2"/>
         <axis xyz="0 1 0"/>
-        <origin rpy="0 0 0" xyz="0 0 0.34"/>
-        <limit lower="-${PI/2}" upper="${PI/2}" effort="${effort}" velocity="${velocity}"/>
+        <origin rpy="0 0 0" xyz="0 0 ${link1_length}"/>
+        <limit lower="-${3*PI/4}" upper="${3*PI/4}" effort="${effort}" velocity="${velocity}"/>
+    </joint>
+    <link name="claw_link">
+        <visual>
+            <origin rpy="0 0 0" xyz="0 0 0.01"/>
+            <geometry>
+                <cylinder radius="0.04" length="0.02"/>
+            </geometry>
+        </visual>
+    </link>
+    <joint name="arm_to_claw_joint" type="fixed">
+        <parent link="arm_link_2"/>
+        <child link="claw_link"/>
+        <origin rpy="0 0 0" xyz="0 0 ${link2_length}"/>
+    </joint>
+    <link name="gripper_right">
+        <visual>
+            <origin rpy="0 0 -${PI/2}" xyz="0 -0.02 ${finger_length/2}"/>
+            <geometry>
+                <cylinder radius="0.02" length="${finger_length}"/>
+            </geometry>
+        </visual>
+    </link>
+    <link name="gripper_left">
+    <visual>
+        <origin rpy="0 0 -${PI/2}" xyz="0 0.02 ${finger_length/2}"/>
+        <geometry>
+            <cylinder radius="0.02" length="${finger_length}"/>
+        </geometry>
+    </visual>
+    </link>
+    <joint name="gripper_joint_1" type="revolute">
+        <parent link="claw_link"/>
+        <child link="gripper_right"/>
+        <axis xyz="1 0 0"/>
+        <origin rpy="0 0 0" xyz="0 0 0"/>
+        <limit lower="0" upper="${PI/2}" effort="${effort}" velocity="${velocity}"/>
+    </joint>
+    <joint name="gripper_joint_2" type="revolute">
+        <parent link="claw_link"/>
+        <child link="gripper_left"/>
+        <axis xyz="1 0 0"/>
+        <origin rpy="0 0 0" xyz="0 0 0"/>
+        <limit lower="0" upper="${PI/2}" effort="${effort}" velocity="${velocity}"/>
+        <mimic joint="gripper_joint_1" multiplier="-1"/>
     </joint>
     <!-- Primeiro 6cm, depois 34cm, depois 27cm -->
 </robot>
+<!-- <ros2_control name="TheseusSystem" type="system">
+    <hardware>
+        <plugin>mock_components/GenericSystem</plugin>
+        <param name="example_param">example_value</param>
+    </hardware>
+    <!-- Arm joints -->
+    <joint name="arm_joint_1">
+        <command_interface name="position"/>
+        <state_interface name="position"/>
+    </joint>
+    <joint name="arm_joint_2">
+        <command_interface name="position"/>
+        <state_interface name="position"/>
+    </joint>
+    <!-- Gripper joint -->
+    <joint name="gripper_joint_1">
+        <command_interface name="position"/>
+        <state_interface name="position"/>
+    </joint>
+</ros2_control> -->

Commit message: gazebo working. hardware interface with problems in ros2_control plus libserial

File: theseus_description/urdf/theseus.urdf.xacro (robot description, xacro)
@@ -1,4 +1,12 @@
 <?xml version="1.0"?>
 <robot xmlns:xacro="http://www.ros.org/wiki/xacro" name="utbots_manipulator">
+    <!-- TODO Adjust all links, joints, visuals, collision and inertias for theseus -->
+    <xacro:arg name="is_sim" default="false" />
+    <xacro:arg name="is_ignition" default="true" />
+    <!-- Include Gazebo Parameters (only relevant for sim) -->
+    <xacro:include filename="$(find theseus_description)/urdf/theseus_gazebo.xacro"/>
+    <!-- Include ros2_control plugins -->
+    <xacro:include filename="$(find theseus_description)/urdf/theseus_ros2_control.xacro"/>
+    <!-- Useful XACRO variables -->
     <xacro:property name="PI" value="3.14159265358979323846"/>
     <xacro:property name="effort" value="10.0"/>
@@ -7,6 +15,17 @@
     <xacro:property name="link2_length" value="0.27"/>
     <xacro:property name="finger_length" value="0.15"/>
+    <!-- Macros -->
+    <xacro:macro name="default_inertial" params="mass">
+        <inertial>
+            <mass value="${mass}"/>
+            <inertia ixx="1.0" ixy="0.0" ixz="0.0"
+                     iyy="1.0" iyz="0.0"
+                     izz="1.0"/>
+        </inertial>
+    </xacro:macro>
+    <!-- Links and joints -->
     <link name="world"/>
     <link name="base_link">
+        <xacro:default_inertial mass="1.0"/>
         <visual>
             <origin rpy="0 0 0" xyz="0 0 0.03"/>
@@ -15,4 +34,10 @@
             </geometry>
         </visual>
+        <collision>
+            <origin rpy="0 0 0" xyz="0 0 0.03"/>
+            <geometry>
+                <cylinder radius="0.15" length="0.06"/>
+            </geometry>
+        </collision>
     </link>
     <joint name="base_arm_joint" type="fixed">
@@ -22,4 +47,5 @@
     </joint>
     <link name="arm_link_1">
+        <xacro:default_inertial mass="1.0"/>
         <visual>
             <origin rpy="0 0 0" xyz="0 0 ${link1_length/2}"/>
@@ -28,4 +54,10 @@
             </geometry>
         </visual>
+        <collision>
+            <origin rpy="0 0 0" xyz="0 0 ${link1_length/2}"/>
+            <geometry>
+                <cylinder radius="0.05" length="${link1_length}"/>
+            </geometry>
+        </collision>
     </link>
     <joint name="arm_joint_1" type="revolute">
@@ -37,4 +69,5 @@
     </joint>
      <link name="arm_link_2">
+        <xacro:default_inertial mass="1.0"/>
         <visual>
             <origin rpy="0 0 0" xyz="0 0 ${link2_length/2}"/>
@@ -43,4 +76,10 @@
             </geometry>
         </visual>
+        <collision>
+            <origin rpy="0 0 0" xyz="0 0 ${link2_length/2}"/>
+            <geometry>
+                <cylinder radius="0.05" length="${link2_length}"/>
+            </geometry>
+        </collision>
     </link>
     <joint name="arm_joint_2" type="revolute">
@@ -52,4 +91,5 @@
     </joint>
     <link name="claw_link">
+        <xacro:default_inertial mass="1.0"/>
         <visual>
             <origin rpy="0 0 0" xyz="0 0 0.01"/>
@@ -58,4 +98,10 @@
             </geometry>
         </visual>
+        <collision>
+            <origin rpy="0 0 0" xyz="0 0 0.01"/>
+            <geometry>
+                <cylinder radius="0.04" length="0.02"/>
+            </geometry>
+        </collision>
     </link>
     <joint name="arm_to_claw_joint" type="fixed">
@@ -65,4 +111,5 @@
     </joint>
     <link name="gripper_right">
+        <xacro:default_inertial mass="1.0"/>
         <visual>
             <origin rpy="0 0 -${PI/2}" xyz="0 -0.02 ${finger_length/2}"/>
@@ -71,12 +118,25 @@
             </geometry>
         </visual>
+        <collision>
+            <origin rpy="0 0 -${PI/2}" xyz="0 -0.02 ${finger_length/2}"/>
+            <geometry>
+                <cylinder radius="0.02" length="${finger_length}"/>
+            </geometry>
+        </collision>
     </link>
     <link name="gripper_left">
-    <visual>
-        <origin rpy="0 0 -${PI/2}" xyz="0 0.02 ${finger_length/2}"/>
-        <geometry>
-            <cylinder radius="0.02" length="${finger_length}"/>
-        </geometry>
-    </visual>
+        <xacro:default_inertial mass="1.0"/>
+        <visual>
+            <origin rpy="0 0 -${PI/2}" xyz="0 0.02 ${finger_length/2}"/>
+            <geometry>
+                <cylinder radius="0.02" length="${finger_length}"/>
+            </geometry>
+        </visual>
+        <collision>
+            <origin rpy="0 0 -${PI/2}" xyz="0 -0.02 ${finger_length/2}"/>
+            <geometry>
+                <cylinder radius="0.02" length="${finger_length}"/>
+            </geometry>
+        </collision>
     </link>
     <joint name="gripper_joint_1" type="revolute">
@@ -92,27 +152,7 @@
         <axis xyz="1 0 0"/>
         <origin rpy="0 0 0" xyz="0 0 0"/>
+        <mimic joint="gripper_joint_1" multiplier="-1"/>
         <limit lower="0" upper="${PI/2}" effort="${effort}" velocity="${velocity}"/>
-        <mimic joint="gripper_joint_1" multiplier="-1"/>
     </joint>
     <!-- Primeiro 6cm, depois 34cm, depois 27cm -->
 </robot>
-<!-- <ros2_control name="TheseusSystem" type="system">
-    <hardware>
-        <plugin>mock_components/GenericSystem</plugin>
-        <param name="example_param">example_value</param>
-    </hardware>
-    <!-- Arm joints -->
-    <joint name="arm_joint_1">
-        <command_interface name="position"/>
-        <state_interface name="position"/>
-    </joint>
-    <joint name="arm_joint_2">
-        <command_interface name="position"/>
-        <state_interface name="position"/>
-    </joint>
-    <!-- Gripper joint -->
-    <joint name="gripper_joint_1">
-        <command_interface name="position"/>
-        <state_interface name="position"/>
-    </joint>
-</ros2_control> -->

Commit message: theseus simulation and forward control worked

File: theseus_description/urdf/theseus.urdf.xacro (robot description, xacro)
@@ -22,9 +22,22 @@
     <!-- Mesh scale -->
     <xacro:property name="mesh_scale" value="0.003 0.003 0.003"/>
+    <material name="default_red">
+        <color rgba="0.8 0.2 0.2 1"/>
+    </material>
+    <xacro:macro name="default_sim_texture">
+        <material name="default_red">
+            <ambient>0.4 0.4 0.4 1</ambient>
+            <diffuse>0.8 0.2 0.2 1</diffuse>
+            <specular>0.1 0.1 0.1 1</specular>
+        </material>
+        <gazebo>
+            <cast_shadows>true</cast_shadows>
+        </gazebo>
+    </xacro:macro>
     <!-- Joint distances -->
     <!-- They are relative to one another eg. arm_joint_2 distances are relative to arm_joint_1 position -->
     <xacro:property name="base_arm_joint_x" value="0.0"/>
     <xacro:property name="base_arm_joint_y" value="0.0"/>
-    <xacro:property name="base_arm_joint_z" value="0.0"/>
+    <xacro:property name="base_arm_joint_z" value="0.00"/>
     <xacro:property name="arm_joint_1_x" value="0.0"/>
     <xacro:property name="arm_joint_1_y" value="0.0"/>
@@ -39,8 +52,9 @@
     <xacro:property name="arm_joint_4_y" value="-0.25"/>
     <xacro:property name="arm_joint_4_z" value="-0.91"/>
-    <xacro:property name="gripper_joint_x" value="0.04"/>
+    <xacro:property name="gripper_joint_x" value="0.0"/>
     <xacro:property name="gripper_joint_y" value="0.0"/>
-    <xacro:property name="gripper_joint_z" value="-0.22"/>
-    <xacro:property name="finger_length" value="0.05"/>
+    <xacro:property name="gripper_joint_z" value="-0.12"/>
+    <xacro:property name="finger_length" value="0.14"/>
+    <xacro:property name="finger_separation" value="0.04"/>
     <!-- Links and Joints -->
     <link name="world"/>
@@ -48,11 +62,12 @@
         <xacro:default_inertial mass="0.2"/>
         <visual>
-            <origin rpy="0 0 0" xyz="-0.015 0 0.38"/>
+            <origin rpy="0 0 0" xyz="${base_arm_joint_x-0.015} ${base_arm_joint_y} ${base_arm_joint_z+0.38}"/>
             <geometry>
                 <mesh filename="package://theseus_description/meshes/theseus_link_1.stl" scale="${mesh_scale}"/>
             </geometry>
-        </visual>
-        <collision>
-            <origin rpy="0 0 0" xyz="-0.015 0 0.38"/>
+            <xacro:default_sim_texture/>
+        </visual>
+        <collision>
+            <origin rpy="0 0 0" xyz="${base_arm_joint_x-0.015} ${base_arm_joint_y} ${base_arm_joint_z+0.38}"/>
             <geometry>
                 <mesh filename="package://theseus_description/meshes/theseus_link_1.stl" scale="${mesh_scale}"/>
@@ -63,5 +78,5 @@
         <parent link="world"/>
         <child link="base_link"/>
-        <origin rpy="0 0 0" xyz="0 0 0"/>
+        <origin rpy="0 0 0" xyz="${base_arm_joint_x} ${base_arm_joint_y} ${base_arm_joint_z}"/>
     </joint>
     <link name="arm_link_1">
@@ -73,4 +88,5 @@
                 <mesh filename="package://theseus_description/meshes/theseus_link_2.stl" scale="${mesh_scale}"/>
             </geometry>
+            <xacro:default_sim_texture/>
         </visual>
         <collision>
@@ -96,4 +112,5 @@
                 <mesh filename="package://theseus_description/meshes/theseus_link_3.stl" scale="${mesh_scale}"/>
             </geometry>
+            <xacro:default_sim_texture/>
         </visual>
         <collision>
@@ -120,4 +137,5 @@
                 <mesh filename="package://theseus_description/meshes/theseus_link_4.stl" scale="${mesh_scale}"/>
             </geometry>
+            <xacro:default_sim_texture/>
         </visual>
         <collision>
@@ -143,4 +161,5 @@
                 <mesh filename="package://theseus_description/meshes/theseus_link_5.stl" scale="${mesh_scale}"/>
             </geometry>
+            <xacro:default_sim_texture/>
         </visual>
         <collision>
@@ -166,4 +185,5 @@
                 <mesh filename="package://theseus_description/meshes/gripper_main_link.stl" scale="${mesh_scale}"/>
             </geometry>
+            <xacro:default_sim_texture/>
         </visual>
         <collision>
@@ -188,4 +208,5 @@
                 <mesh filename="package://theseus_description/meshes/gripper_link.stl" scale="${mesh_scale}"/>
             </geometry>
+            <xacro:default_sim_texture/>
         </visual>
         <collision>
@@ -203,4 +224,5 @@
                 <mesh filename="package://theseus_description/meshes/gripper_sub_link.stl" scale="${mesh_scale}"/>
             </geometry>
+            <xacro:default_sim_texture/>
         </visual>
         <collision>
@@ -215,5 +237,5 @@
         <child link="gripper_right"/>
         <axis xyz="0 1 0"/>
-        <origin rpy="0 0 0" xyz="${-gripper_joint_x} ${gripper_joint_y} ${gripper_joint_z}"/>
+        <origin rpy="0 0 0" xyz="${-finger_separation} 0 ${-finger_length}"/>
         <limit lower="${-PI/9}" upper="${PI/2}" effort="${effort}" velocity="${velocity}"/>
     </joint>
@@ -222,5 +244,5 @@
         <child link="gripper_left"/>
         <axis xyz="0 1 0"/>
-        <origin rpy="0 0 0" xyz="${gripper_joint_x} ${gripper_joint_y} ${gripper_joint_z}"/>
+        <origin rpy="0 0 0" xyz="${finger_separation} 0 ${-finger_length}"/>
         <mimic joint="gripper_joint_1" multiplier="-1"/>
         <limit lower="${-PI/9}" upper="${PI/2}" effort="${effort}" velocity="${velocity}"/>

Commit message: model name corrected, but moveit doesnt connect to controllers

File: theseus_description/urdf/theseus.urdf.xacro (robot description, xacro)
@@ -1,4 +1,4 @@
 <?xml version="1.0"?>
-<robot xmlns:xacro="http://www.ros.org/wiki/xacro" name="utbots_manipulator">
+<robot xmlns:xacro="http://www.ros.org/wiki/xacro" name="theseus">
     <!-- Simulation flags for switching simulation engines before and after ROS2 Humble -->
     <xacro:arg name="is_sim" default="false" />

File: theseus_description/urdf/theseus_ros2_control.xacro (robot description, xacro)
@@ -1,6 +1,7 @@
 <?xml version="1.0"?>
-<robot xmlns:xacro="http://www.ros.org/wiki/xacro" name="utbots_manipulator">
+<robot xmlns:xacro="http://www.ros.org/wiki/xacro" name="theseus">
     <ros2_control name="ManipulatorSystem" type="system">
         <xacro:property name="PI" value="3.14159265358979323846"/>
+        <xacro:property name="initial_positions" value="$(find theseus_moveit)/config/initial_positions.yaml"/>
         <!-- ros2_control Gazebo only -->
         <xacro:if value="$(arg is_sim)">

File: theseus_moveit/config/theseus.ros2_control(onlyref_to_remove).xacro (robot description, xacro)
@@ -1,5 +1,5 @@
 <?xml version="1.0"?>
 <robot xmlns:xacro="http://www.ros.org/wiki/xacro">
-    <xacro:macro name="utbots_manipulator_ros2_control" params="name initial_positions_file">
+    <xacro:macro name="theseus_ros2_control" params="name initial_positions_file">
         <xacro:property name="initial_positions" value="${load_yaml(initial_positions_file)['initial_positions']}"/>
         <ros2_control name="${name}" type="system">
@@ -13,5 +13,4 @@
                   <param name="initial_value">${initial_positions['arm_joint_1']}</param>
                 </state_interface>
-                <state_interface name="velocity"/>
             </joint>
             <joint name="arm_joint_2">
@@ -20,5 +19,4 @@
                   <param name="initial_value">${initial_positions['arm_joint_2']}</param>
                 </state_interface>
-                <state_interface name="velocity"/>
             </joint>
             <joint name="arm_joint_3">
@@ -27,5 +25,4 @@
                   <param name="initial_value">${initial_positions['arm_joint_3']}</param>
                 </state_interface>
-                <state_interface name="velocity"/>
             </joint>
             <joint name="arm_joint_4">
@@ -34,5 +31,4 @@
                   <param name="initial_value">${initial_positions['arm_joint_4']}</param>
                 </state_interface>
-                <state_interface name="velocity"/>
             </joint>
             <joint name="gripper_joint">
@@ -41,5 +37,4 @@
                   <param name="initial_value">${initial_positions['gripper_joint']}</param>
                 </state_interface>
-                <state_interface name="velocity"/>
             </joint>
             <joint name="gripper_joint_1">
@@ -48,5 +43,4 @@
                   <param name="initial_value">${initial_positions['gripper_joint_1']}</param>
                 </state_interface>
-                <state_interface name="velocity"/>
             </joint>
         </ros2_control>

Commit message: functional goal in theseus

File: theseus_description/urdf/theseus.urdf.xacro (robot description, xacro)
@@ -18,5 +18,5 @@
         </inertial>
     </xacro:macro>
-    <xacro:property name="effort" value="10.0"/>
+    <xacro:property name="effort" value="200.0"/>
     <xacro:property name="velocity" value="5.0"/>
     <!-- Mesh rendering properties -->
